File: kulinski.sch (KiCad schematic (older format))
At the start: 22 parts

Commit message: schema all elements
Parts:
- C? (x2): value C -> u1
- C?: value CP -> 2u2
- R? (x2): value R -> 1k
- R?: value R -> 2k7
- R? (x3): value R -> k47
- R?: value R -> 47k
- R?: value R -> k12
- R?: value R -> k91
- R?: value RTRIM -> 5k
Connections:
- wire segments 22 -> 21
Other:
- moved on the sheet: C?, D?, R?
Changed lines of the file:
@@
 L Device:R R?
 U 1 1 5D1A9D87
-P 1900 5000
-F 0 "R?" H 1970 5046 50  0000 L CNN
-F 1 "R" H 1970 4955 50  0000 L CNN
-F 2 "" V 1830 5000 50  0001 C CNN
-F 3 "~" H 1900 5000 50  0001 C CNN
-	1    1900 5000
+P 1800 5900
+F 0 "R?" H 1870 5946 50  0000 L CNN
+F 1 "1k" H 1870 5855 50  0000 L CNN
+F 2 "" V 1730 5900 50  0001 C CNN
+F 3 "~" H 1800 5900 50  0001 C CNN
+	1    1800 5900
 	1    0    0    -1
 $EndComp
@@
 U 1 1 5D1AA05A
 P 2900 4350
-F 0 "R?" H 2970 4396 50  0000 L CNN
-F 1 "R" H 2970 4305 50  0000 L CNN
+F 0 "R?" V 3107 4350 50  0000 C CNN
+F 1 "2k7" V 3016 4350 50  0000 C CNN
 F 2 "" V 2830 4350 50  0001 C CNN
 F 3 "~" H 2900 4350 50  0001 C CNN
@@
 L Device:R R?
 U 1 1 5D1AA329
-P 4000 3800
-F 0 "R?" H 4070 3846 50  0000 L CNN
-F 1 "R" H 4070 3755 50  0000 L CNN
-F 2 "" V 3930 3800 50  0001 C CNN
-F 3 "~" H 4000 3800 50  0001 C CNN
-	1    4000 3800
+P 5050 4050
+F 0 "R?" H 5120 4096 50  0000 L CNN
+F 1 "k47" H 5120 4005 50  0000 L CNN
+F 2 "" V 4980 4050 50  0001 C CNN
+F 3 "~" H 5050 4050 50  0001 C CNN
+	1    5050 4050
 	1    0    0    -1
 $EndComp
@@
 L Device:R R?
 U 1 1 5D1AAA03
-P 4000 4450
-F 0 "R?" H 4070 4496 50  0000 L CNN
-F 1 "R" H 4070 4405 50  0000 L CNN
-F 2 "" V 3930 4450 50  0001 C CNN
-F 3 "~" H 4000 4450 50  0001 C CNN
-	1    4000 4450
+P 5050 4550
+F 0 "R?" H 5120 4596 50  0000 L CNN
+F 1 "k47" H 5120 4505 50  0000 L CNN
+F 2 "" V 4980 4550 50  0001 C CNN
+F 3 "~" H 5050 4550 50  0001 C CNN
+	1    5050 4550
 	1    0    0    -1
 $EndComp
@@
 L Device:R R?
 U 1 1 5D1AABF0
-P 5700 4550
-F 0 "R?" H 5770 4596 50  0000 L CNN
-F 1 "R" H 5770 4505 50  0000 L CNN
-F 2 "" V 5630 4550 50  0001 C CNN
-F 3 "~" H 5700 4550 50  0001 C CNN
-	1    5700 4550
+P 5700 4750
+F 0 "R?" H 5770 4796 50  0000 L CNN
+F 1 "k47" H 5770 4705 50  0000 L CNN
+F 2 "" V 5630 4750 50  0001 C CNN
+F 3 "~" H 5700 4750 50  0001 C CNN
+	1    5700 4750
 	1    0    0    -1
 $EndComp
@@
 L Device:R R?
 U 1 1 5D1AAD08
-P 6550 4550
-F 0 "R?" H 6620 4596 50  0000 L CNN
-F 1 "R" H 6620 4505 50  0000 L CNN
-F 2 "" V 6480 4550 50  0001 C CNN
-F 3 "~" H 6550 4550 50  0001 C CNN
-	1    6550 4550
+P 6550 4750
+F 0 "R?" H 6620 4796 50  0000 L CNN
+F 1 "47k" H 6620 4705 50  0000 L CNN
+F 2 "" V 6480 4750 50  0001 C CNN
+F 3 "~" H 6550 4750 50  0001 C CNN
+	1    6550 4750
 	1    0    0    -1
 $EndComp
@@
 L Device:R R?
 U 1 1 5D1AB35B
-P 7000 4850
-F 0 "R?" H 7070 4896 50  0000 L CNN
-F 1 "R" H 7070 4805 50  0000 L CNN
-F 2 "" V 6930 4850 50  0001 C CNN
-F 3 "~" H 7000 4850 50  0001 C CNN
-	1    7000 4850
+P 6850 4750
+F 0 "R?" H 6920 4796 50  0000 L CNN
+F 1 "1k" H 6920 4705 50  0000 L CNN
+F 2 "" V 6780 4750 50  0001 C CNN
+F 3 "~" H 6850 4750 50  0001 C CNN
+	1    6850 4750
 	1    0    0    -1
 $EndComp
@@
 P 4250 6150
 F 0 "R?" H 4320 6196 50  0000 L CNN
-F 1 "R" H 4320 6105 50  0000 L CNN
+F 1 "k12" H 4320 6105 50  0000 L CNN
 F 2 "" V 4180 6150 50  0001 C CNN
 F 3 "~" H 4250 6150 50  0001 C CNN
@@
 P 4950 6150
 F 0 "R?" H 5020 6196 50  0000 L CNN
-F 1 "R" H 5020 6105 50  0000 L CNN
+F 1 "k91" H 5020 6105 50  0000 L CNN
 F 2 "" V 4880 6150 50  0001 C CNN
 F 3 "~" H 4950 6150 50  0001 C CNN
@@
 P 5700 6200
 F 0 "R?" H 5828 6246 50  0000 L CNN
-F 1 "RTRIM" H 5828 6155 50  0000 L CNN
+F 1 "5k" H 5828 6155 50  0000 L CNN
 F 2 "" V 5630 6200 50  0001 C CNN
 F 3 "~" H 5700 6200 50  0001 C CNN
@@
 L Device:LED D?
 U 1 1 5D1BC838
-P 1900 4400
-F 0 "D?" V 1847 4478 50  0000 L CNN
-F 1 "LED" V 1938 4478 50  0000 L CNN
-F 2 "" H 1900 4400 50  0001 C CNN
-F 3 "~" H 1900 4400 50  0001 C CNN
-	1    1900 4400
-	0    1    1    0
+P 1800 5400
+F 0 "D?" V 1839 5283 50  0000 R CNN
+F 1 "LED" V 1748 5283 50  0000 R CNN
+F 2 "" H 1800 5400 50  0001 C CNN
+F 3 "~" H 1800 5400 50  0001 C CNN
+	1    1800 5400
+	0    -1   -1   0
 $EndComp
 $Comp
@@
 L Device:C C?
 U 1 1 5D1C59A4
-P 3550 4300
-F 0 "C?" V 3298 4300 50  0000 C CNN
-F 1 "C" V 3389 4300 50  0000 C CNN
-F 2 "" H 3588 4150 50  0001 C CNN
-F 3 "~" H 3550 4300 50  0001 C CNN
-	1    3550 4300
+P 4050 4150
+F 0 "C?" V 3798 4150 50  0000 C CNN
+F 1 "u1" V 3889 4150 50  0000 C CNN
+F 2 "" H 4088 4000 50  0001 C CNN
+F 3 "~" H 4050 4150 50  0001 C CNN
+	1    4050 4150
 	0    1    1    0
 $EndComp
@@
 L Device:C C?
 U 1 1 5D1C60C6
-P 3550 4650
-F 0 "C?" V 3298 4650 50  0000 C CNN
-F 1 "C" V 3389 4650 50  0000 C CNN
-F 2 "" H 3588 4500 50  0001 C CNN
-F 3 "~" H 3550 4650 50  0001 C CNN
-	1    3550 4650
+P 4050 4500
+F 0 "C?" V 3798 4500 50  0000 C CNN
+F 1 "u1" V 3889 4500 50  0000 C CNN
+F 2 "" H 4088 4350 50  0001 C CNN
+F 3 "~" H 4050 4500 50  0001 C CNN
+	1    4050 4500
 	0    1    1    0
 $EndComp
@@
 L Diode:1N4148 D?
 U 1 1 5D1C76C5
-P 7050 3850
-F 0 "D?" V 7004 3929 50  0000 L CNN
-F 1 "1N4148" V 7095 3929 50  0000 L CNN
-F 2 "Diode_THT:D_DO-35_SOD27_P7.62mm_Horizontal" H 7050 3675 50  0001 C CNN
-F 3 "https://assets.nexperia.com/documents/data-sheet/1N4148_1N4448.pdf" H 7050 3850 50  0001 C CNN
-	1    7050 3850
+P 6850 4100
+F 0 "D?" V 6804 4179 50  0000 L CNN
+F 1 "1N4148" V 6895 4179 50  0000 L CNN
+F 2 "Diode_THT:D_DO-35_SOD27_P7.62mm_Horizontal" H 6850 3925 50  0001 C CNN
+F 3 "https://assets.nexperia.com/documents/data-sheet/1N4148_1N4448.pdf" H 6850 4100 50  0001 C CNN
+	1    6850 4100
 	0    1    1    0
 $EndComp
@@
 L Diode:1N4148 D?
 U 1 1 5D1C8D81
-P 7350 3850
-F 0 "D?" V 7304 3929 50  0000 L CNN
-F 1 "1N4148" V 7395 3929 50  0000 L CNN
-F 2 "Diode_THT:D_DO-35_SOD27_P7.62mm_Horizontal" H 7350 3675 50  0001 C CNN
-F 3 "https://assets.nexperia.com/documents/data-sheet/1N4148_1N4448.pdf" H 7350 3850 50  0001 C CNN
-	1    7350 3850
+P 7150 4100
+F 0 "D?" V 7104 4179 50  0000 L CNN
+F 1 "1N4148" V 7195 4179 50  0000 L CNN
+F 2 "Diode_THT:D_DO-35_SOD27_P7.62mm_Horizontal" H 7150 3925 50  0001 C CNN
+F 3 "https://assets.nexperia.com/documents/data-sheet/1N4148_1N4448.pdf" H 7150 4100 50  0001 C CNN
+	1    7150 4100
 	0    1    1    0
 $EndComp
@@
 L Diode:BZX84Cxx D?
 U 1 1 5D1CB1BD
-P 2900 3700
-F 0 "D?" V 2854 3779 50  0000 L CNN
-F 1 "BZX84Cxx" V 2945 3779 50  0000 L CNN
-F 2 "Diode_SMD:D_SOT-23_ANK" H 2900 3525 50  0001 C CNN
-F 3 "https://diotec.com/tl_files/diotec/files/pdf/datasheets/bzx84c2v4.pdf" H 2900 3700 50  0001 C CNN
-	1    2900 3700
+P 4550 4300
+F 0 "D?" V 4504 4379 50  0000 L CNN
+F 1 "BZX84Cxx" V 4595 4379 50  0000 L CNN
+F 2 "Diode_SMD:D_SOT-23_ANK" H 4550 4125 50  0001 C CNN
+F 3 "https://diotec.com/tl_files/diotec/files/pdf/datasheets/bzx84c2v4.pdf" H 4550 4300 50  0001 C CNN
+	1    4550 4300
 	0    1    1    0
 $EndComp
@@
 P 4600 6150
 F 0 "C?" H 4718 6196 50  0000 L CNN
-F 1 "CP" H 4718 6105 50  0000 L CNN
+F 1 "2u2" H 4718 6105 50  0000 L CNN
 F 2 "" H 4638 6000 50  0001 C CNN
 F 3 "~" H 4600 6150 50  0001 C CNN
@@
 $EndComp
 Wire Wire Line
-	6550 5550 6550 6500
-Wire Wire Line
 	1800 6750 1800 6500
 Wire Wire Line
@@
 Connection ~ 2850 6500
 Wire Wire Line
-	6550 5250 6550 4700
-Wire Wire Line
-	5700 4700 5700 5150
-Wire Wire Line
 	5700 5600 4250 5600
 Wire Wire Line
 	5700 5550 5700 5600
-Connection ~ 5700 5600
-Wire Wire Line
-	5700 5600 5700 5750
 Wire Wire Line
 	2850 6500 3650 6500
@@
 Wire Wire Line
 	4250 5600 3950 5600
+Wire Wire Line
+	5700 5150 5700 4900
+Wire Wire Line
+	6550 5250 6550 4900
+Wire Wire Line
+	6550 5550 6550 6500
 $EndSCHEMATC
